File: MicErgo_left/MicErgo_left.kicad_sch (KiCad schematic)
At the start: 68 parts, among them J1 MJ-4PP-9, SW00 SW_Push, SW1 SW_Push, SW10 SW_Push, SW11 SW_Push, SW12 SW_Push, SW13 SW_Push, SW14 SW_Push, SW15 SW_Push, SW16 SW_Push, SW17 SW_Push, SW18 SW_Push, SW19 SW_Push, SW2 SW_Push, SW20 SW_Push, SW21 SW_Push, SW22 SW_Push, SW23 SW_Push, SW24 SW_Push, SW25 SW_Push, SW26 RotaryEncoder_Switch, SW27 SW_Push, SW28 SW_Push, SW29 SW_Push, SW3 SW_Push, SW30 SW_Push, SW31 SW_Push, SW32 SW_Push, SW4 SW_Push, SW5 SW_Push, SW6 SW_Push, SW7 SW_Push, SW8 SW_Push, SW9 SW_Push, U1 ProMicro

Commit message: Add files via upload
Parts:
- removed D32: D, kbd_Parts:Diode_SMD, symbol Device:D
- removed J1: MJ-4PP-9, kbd_Parts:TRRS_MJ-4PP-9, symbol kbd:MJ-4PP-9
- removed SW32: SW_Push, kbd_SW_PCBA:Choc_v2_Hotswap_1u_Narrow, symbol Switch:SW_Push
- added D26, D33, D34: D, my_foot:Diode_SMD_top, symbol Device:D
- added J1: TRRS_MJ-4PP-9(acid_mmVer), kbd_Parts:TRRS_MJ-4PP-9, symbol kbd:TRRS_MJ-4PP-9(acid_mmVer)
- added SW26: SW_Push, my_foot:Choc_v2_Hotswap_1u_Narrow, symbol Switch:SW_Push
- added SW33, SW34: SW_Push, kbd_SW_PCBA:Choc_v2_予備用, symbol Switch:SW_Push
- D1, D10, D11, D12, D13, D14, D15, D16, D17, D18, D19, D2, D20, D21, D22, D23, D24, D25, D27, D28, D29, D3, D30, D31, D4, D5, D6, D7, D8, D9: footprint kbd_Parts:Diode_SMD -> my_foot:Diode_SMD_top
- D32: renamed from D26; footprint kbd_Parts:Diode_SMD -> my_foot:Diode_SMD_top
- SW1, SW10, SW11, SW12, SW13, SW14, SW15, SW16, SW17, SW18, SW19, SW2, SW20, SW21, SW22, SW23, SW24, SW25, SW27, SW28, SW29, SW3, SW30, SW31, SW4, SW5, SW6, SW7, SW8, SW9: footprint kbd_SW_PCBA:Choc_v2_Hotswap_1u_Narrow -> my_foot:Choc_v2_Hotswap_1u_Narrow
- renumbered SW26 to SW32
Connections:
- net DATA: now also J1.B
- net GND: now also J1.A
- net VCC: now also J1.D
- net col0: now also SW25.1
- net col1: now also SW26.1
- net col2: now also SW27.1
- net col3: now also SW28.1
- net col4: now also SW29.1
- net col5: now also SW30.1
- net col6: now also SW31.1, SW33.1, SW34.1; no longer SW25.1, SW27.1, SW28.1
- net roA: now also U1.13 (B6/10); no longer U1.11 (8/B4)
- net row0: now also D31.1 (K); no longer D25.1 (K), D29.1 (K)
- net row1: no longer D30.1 (K)
- net row2: now also D33.1 (K); no longer D27.1 (K), D31.1 (K)
- net row3: now also D34.1 (K); no longer D28.1 (K)
- removed net col7: SW29.1, SW30.1, SW31.1, U1.13 (B6/10)
- new net: D26.2 (A), SW26.2
- new net: D34.2 (A), SW34.2
- new net: D33.2 (A), SW33.2
- new net row4: D25.1 (K), D26.1 (K), D27.1 (K), D28.1 (K), D29.1 (K), D30.1 (K), U1.11 (8/B4)
Other:
- moved on the sheet: D25, D27, D28, D29, D30, D31, D32, SW25, SW27, SW28, SW29, SW30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
